Commit message: handle

File: assets/gapartnet_example/11304/mobility_annotation_gapartnet.urdf (robot description, URDF)
Before this commit: robot partnet_b5b34464d1270673617724635ed7cc4b, 6 links, 5 joints
Links:
- link link_3: geometry collision mesh filename=textured_objs/original-2.obj scale=1.5 2.0 1.0; visual mesh filename=textured_objs/original-2.obj
- link link_4: geometry collision mesh filename=textured_objs/original-17.obj scale=1.5 2.0 1.0; visual mesh filename=textured_objs/original-17.obj

File: assets/gapartnet_example/11712/mobility_annotation_gapartnet.urdf (robot description, URDF)
Before this commit: robot partnet_f7e0a103c97469d5a168e247bb97e471, 6 links, 5 joints
Links:
- link link_3: geometry collision mesh filename=textured_objs/modified-0-original-13.obj scale=1.5 2.0 1.0; collision mesh filename=textured_objs/modified-0-original-14.obj scale=1.5 2.0 1.0
- link link_4: geometry collision mesh filename=textured_objs/modified-0-original-7.obj scale=1.5 2.0 1.0; collision mesh filename=textured_objs/modified-0-original-8.obj scale=1.5 2.0 1.0

File: assets/gapartnet_example/45661/mobility_annotation_gapartnet.urdf (robot description, URDF)
Before this commit: robot partnet_2b37f9944a63ba4b4c3aee8e9d3a6ffa, 8 links, 7 joints
Links:
- link link_4: geometry collision mesh filename=textured_objs/original-38.obj scale=1.5 2.0 1.0; collision mesh filename=textured_objs/original-39.obj scale=1.5 2.0 1.0
- link link_5: geometry collision mesh filename=textured_objs/original-30.obj scale=1.5 2.0 1.0; collision mesh filename=textured_objs/original-31.obj scale=1.5 2.0 1.0
- link link_6: geometry collision mesh filename=textured_objs/original-54.obj scale=1.5 2.0 1.0; collision mesh filename=textured_objs/original-55.obj scale=1.5 2.0 1.0
